File: neural_net_demo_board/neural_net_demo_board.kicad_sch (KiCad schematic)
At the start: 36 parts, among them J1 USB_C_Receptacle_USB2.0_16P, U1 XIAO-RP2040-DIP, U2 TMP36GRTZ-REEL7, U3 TEMT6000X01, U4 MCU_RaspberryPi_RP2040_RP2040, U5 NCP1117-3.3_SOT223, Y1 ABM8-272-T3

Commit message: Integrate rp2040, input/outputs
Parts:
- removed U1: XIAO-RP2040-DIP, ScottoKeebs_MCU:Seeed_XIAO_RP2040, symbol Seeed_Studio_XIAO_Series:XIAO-RP2040-DIP
- added C16: 100n, Capacitor_SMD:C_0402_1005Metric, symbol Device:C
- added CONN01x2: Conn_01x02 USB_BOOT, Connector_PinHeader_1.00mm:PinHeader_1x02_P1.00mm_Vertical, symbol Connector_Generic:Conn_01x02
- added D10, D11, D12, D13, D14, D15, D16, D17, D18, D19, D20, D5, D6, D7, D8, D9: SK6812MINI, LED_SMD:LED_SK6812MINI_PLCC4_3.5x3.5mm_P1.75mm, symbol LED:SK6812MINI
- added FLASH1: W25Q128JVS, Package_SO:SOIC-8_5.23x5.23mm_P1.27mm, symbol Memory_Flash:W25Q128JVS
- added R7, R9: 1 kΩ, Resistor_SMD:R_0402_1005Metric, symbol Device:R
- added R8: DO NOT FIT, Resistor_SMD:R_0402_1005Metric, symbol Device:R
- C10, C11, C12, C13, C14, C15, C3, C4, C5, C6, C7, C8, C9: footprint Capacitor_SMD:C_0805_2012Metric -> Capacitor_SMD:C_0402_1005Metric
- R1, R2, R3, R4, R5, R6: footprint (none) -> Resistor_SMD:R_0402_1005Metric
- RP2040: renamed from U4; footprint RP2040_minimal:RP2040-QFN-56 -> RP2040_minimal_r2:RP2040-QFN-56
- USB-C1: renamed from J1; footprint (none) -> Connector_USB:USB_C_Receptacle_GCT_USB4105-xx-A_16P_TopMnt_Horizontal
- renumbered U3 to AMB.LIGHT1, Y1 to OSC.1, U2 to TEMP1
Connections:
- net +3V3 is gone; now on net +3.3V: C10.1, C2.1, C3.1, C4.1, C5.1, C6.1, C7.1, C8.1, C9.1, RP2040.1 (IOVDD), RP2040.10 (IOVDD), RP2040.22 (IOVDD), RP2040.33 (IOVDD), RP2040.42 (IOVDD), RP2040.43 (ADC_AVDD), RP2040.44 (VREG_IN), RP2040.48 (USB_VDD), RP2040.49 (IOVDD), U5.2 (VO)
- net +3.3V: now also C16.1, D10.4 (VDD), D11.4 (VDD), D12.4 (VDD), D13.4 (VDD), D14.4 (VDD), D15.4 (VDD), D16.4 (VDD), D17.4 (VDD), D18.4 (VDD), D19.4 (VDD), D20.4 (VDD), D5.4 (VDD), D6.4 (VDD), D7.4 (VDD), D8.4 (VDD), D9.4 (VDD), FLASH1.8 (VCC), R8.2
- net COL 1: now also RP2040.28 (GPIO17)
- net COL 2: now also RP2040.37 (GPIO25)
- net COL 3: now also RP2040.38 (GPIO26_ADC0)
- net COL 4: now also RP2040.39 (GPIO27_ADC1)
- net CRYSTAL OUT: now also R9.2; no longer C15.2, OSC.1.3
- net GND: now also C16.2, CONN01x2.2 (Pin_2), D10.2 (VSS), D11.2 (VSS), D12.2 (VSS), D13.2 (VSS), D14.2 (VSS), D15.2 (VSS), D16.2 (VSS), D17.2 (VSS), D18.2 (VSS), D19.2 (VSS), D20.2 (VSS), D5.2 (VSS), D6.2 (VSS), D7.2 (VSS), D8.2 (VSS), D9.2 (VSS), FLASH1.4 (GND)
- net LIGHT OUT: now also RP2040.40 (GPIO28_ADC2)
- net RGB: now also RP2040.14 (GPIO11)
- net ROW 1: now also RP2040.29 (GPIO18)
- net TEMP OUT: now also RP2040.41 (GPIO29_ADC3)
- net RGB2: now reaches RP2040.15 (GPIO12)
- net RGB2: now also D5.3 (DIN)
- net QSPI_SD3: now reaches RP2040.51 (QSPI_SD3)
- net QSPI_SD3: now also FLASH1.7 (IO3)
- net QSPI_SCLK: now reaches RP2040.52 (QSPI_SCLK)
- net QSPI_SCLK: now also FLASH1.6 (CLK)
- net QSPI_SD0: now reaches RP2040.53 (QSPI_SD0)
- net QSPI_SD0: now also FLASH1.5 (DI(IO0))
- net QSPI_SD2: now reaches RP2040.54 (QSPI_SD2)
- net QSPI_SD2: now also FLASH1.3 (IO2)
- net QSPI_SD1: now reaches RP2040.55 (QSPI_SD1)
- net QSPI_SD1: now also FLASH1.2 (DO(IO1))
- net QSPI_SS: now reaches RP2040.56 (QSPI_SS)
- net QSPI_SS: now also FLASH1.1 (~{CS}), R7.2, R8.1
- new net: D15.1 (DOUT), D16.3 (DIN)
- new net: D14.1 (DOUT), D15.3 (DIN)
- new net: D19.1 (DOUT), D20.3 (DIN)
- new net: D11.1 (DOUT), D12.3 (DIN)
- new net: D10.1 (DOUT), D11.3 (DIN)
- new net: CONN01x2.1 (Pin_1), R7.1
- new net: C15.2, OSC.1.3, R9.1
- new net: D5.1 (DOUT), D6.3 (DIN)
- new net: D8.1 (DOUT), D9.3 (DIN)
- new net: D7.1 (DOUT), D8.3 (DIN)
- new net: D13.1 (DOUT), D14.3 (DIN)
- new net: D18.1 (DOUT), D19.3 (DIN)
- new net: D17.1 (DOUT), D18.3 (DIN)
- new net: D16.1 (DOUT), D17.3 (DIN)
- new net: D6.1 (DOUT), D7.3 (DIN)
- new net: D12.1 (DOUT), D13.3 (DIN)
- new net: D10.3 (DIN), D9.1 (DOUT)
Other:
- moved on the sheet: R5

Commit message: pcb's basically done atp
Parts:
- added C17: 10u, Capacitor_SMD:C_0805_2012Metric, symbol Device:C
- added CONN01x24: Conn_01x24, Connector_PinHeader_1.00mm:PinHeader_1x24_P1.00mm_Vertical, symbol Connector_Generic:Conn_01x24
Connections:
- net +3.3V: now also C17.1
- net GND: now also C17.2
- net GP2: now reaches RP2040.11 (GPIO8)
- net GP2: now also CONN01x24.9 (Pin_9)
- net GP1: now reaches RP2040.12 (GPIO9)
- net GP1: now also CONN01x24.10 (Pin_10)
- net GP0: now reaches RP2040.13 (GPIO10)
- net GP0: now also CONN01x24.11 (Pin_11)
- net GP13: now reaches RP2040.16 (GPIO13)
- net GP13: now also CONN01x24.12 (Pin_12)
- net GP14: now reaches RP2040.17 (GPIO14)
- net GP14: now also CONN01x24.13 (Pin_13)
- net GP15: now reaches RP2040.18 (GPIO15)
- net GP15: now also CONN01x24.14 (Pin_14)
- net GP10: now reaches RP2040.2 (GPIO0)
- net GP10: now also CONN01x24.1 (Pin_1)
- net SWCLK: now reaches RP2040.24 (SWCLK)
- net SWCLK: now also CONN01x24.15 (Pin_15)
- net SWD: now reaches RP2040.25 (SWD)
- net SWD: now also CONN01x24.16 (Pin_16)
- net RUN: now reaches RP2040.26 (RUN)
- net RUN: now also CONN01x24.17 (Pin_17)
- net GP16: now reaches RP2040.27 (GPIO16)
- net GP16: now also CONN01x24.18 (Pin_18)
- net GP9: now reaches RP2040.3 (GPIO1)
- net GP9: now also CONN01x24.2 (Pin_2)
- net GP19: now reaches RP2040.30 (GPIO19)
- net GP19: now also CONN01x24.19 (Pin_19)
- net GP20: now reaches RP2040.31 (GPIO20)
- net GP20: now also CONN01x24.20 (Pin_20)
- net GP21: now reaches RP2040.32 (GPIO21)
- net GP21: now also CONN01x24.21 (Pin_21)
- net GP22: now reaches RP2040.34 (GPIO22)
- net GP22: now also CONN01x24.22 (Pin_22)
- net GP23: now reaches RP2040.35 (GPIO23)
- net GP23: now also CONN01x24.23 (Pin_23)
- net GP24: now reaches RP2040.36 (GPIO24)
- net GP24: now also CONN01x24.24 (Pin_24)
- net GP8: now reaches RP2040.4 (GPIO2)
- net GP8: now also CONN01x24.3 (Pin_3)
- net GP7: now reaches RP2040.5 (GPIO3)
- net GP7: now also CONN01x24.4 (Pin_4)
- net GP6: now reaches RP2040.6 (GPIO4)
- net GP6: now also CONN01x24.5 (Pin_5)
- net GP5: now reaches RP2040.7 (GPIO5)
- net GP5: now also CONN01x24.6 (Pin_6)
- net GP4: now reaches RP2040.8 (GPIO6)
- net GP4: now also CONN01x24.7 (Pin_7)
- net GP3: now reaches RP2040.9 (GPIO7)
- net GP3: now also CONN01x24.8 (Pin_8)
Other:
- moved on the sheet: AMB.LIGHT1, C1, C14, C15, C16, C2, CONN01x2, D1, D10, D11, D12, D13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
