File: rp2040-logic-demo-board/rp2040-logic-demo-board.kicad_pcb (KiCad board)
At the start: 2 copper layers, 93.6 x 99 mm, 69 parts, among them U5 NCP1117-3.3_SOT223

Commit message: create 2 files and update 1 file
Parts:
- removed the G*** at (153.9, 59.5)
- removed the G*** at (173.8, 120.8)
- added G***: LOGO, LOGO, B.Cu at (173.8, 121.1)
Other:
- board text added: "Built on RP2040. Powered by MicroPython."
- board text added: "github.com/sidsenthilexe/rp2040-logic-demo-board"
- board text removed: "Built on RP2040 Powered by MicroPython Trained with TensorFlow"
- board text removed: "github.com/sidsenthilexe/neural-net-demo-board"
